File: xmos_avb_brd_V4.brd (EAGLE design)
At the start: 80 x 40 mm, 147 parts, among them IC1 IS25LP080D-JULE-TR_IS25LP080D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, IC3 KSZ9131RNXI-TR, J1 0826-1X1T-KL-F_0826-1X1T-KL-F, J3 ESHF-110-01-L-D-TH, U1 AG9900_AG9905LP, U10 ST-MICROELECTRONICS2_ST1S06PUR, U2 AR8035_AR8035-AL1A-R, U3 XE216-512-TQ128-C20_XE216-512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, U4 ADM1085AKSZ-REEL7_ADM1085AKSZ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, U5 NC7WZ07P6X_NC7WZ07P6X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

Commit message: resolved DRC errors and exported manufacturing data for V4.
Parts:
- removed IC3: KSZ9131RNXI-TR, KSZ9131RNXI-TR:QFN50P700X700X90-49N
- removed R19: 43R2, xmos_avb_brd_V4:RCL_R0402
- moved C58 97.1 mm to (26.1, 27.9), turned to 180 degrees
- moved C57 89.4 mm to (26.1, 25.5), turned to 180 degrees
- moved C56 88.2 mm to (26.1, 30.3), turned to 180 degrees
- moved C30 85.0 mm to (26.1, 32.8), turned to 180 degrees
- moved C9 81.6 mm to (26.0, 35.1), turned to 180 degrees
Connections:
- removed net USB_DM_N: J3.20, U3.47
- removed net USB_DP_P: J3.19, U3.46
- removed net USB_ID: J3.17, U3.43
- removed net USB_RTUNE: R19.2, U3.48
- removed net USB_VBUS: J3.16, U3.45
- net GND: no longer R19.1
Routing:
- net GND: track 86.1 -> 103.0 mm, vias 109 -> 114
- net 3V3_PG: track 0.00 -> 11.9 mm, vias 0 -> 1
- net VDC: track 30.5 -> 40.7 mm
- net VC12: track 12.7 -> 22.6 mm
- net SCL: track 28.8 -> 19.6 mm
- net VC45: track 21.4 -> 30.0 mm
- net SDA: track 25.5 -> 18.4 mm
- net USB_ID: track 5.40 -> 0.00 mm, vias 1 -> 0
- net USB_DP_P: track 5.29 -> 0.00 mm
- net USB_DM_N: track 4.88 -> 0.00 mm
- net USB_RTUNE: track 3.99 -> 0.00 mm, vias 1 -> 0
- net 1V0: track 63.5 -> 67.2 mm, vias 19 -> 20
- net USB_VBUS: track 3.26 -> 0.00 mm, vias 1 -> 0
- net VC1+: track 20.5 -> 22.9 mm
- net PHY_RSTN: track 27.0 -> 28.8 mm
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