File: xmos_avb_brd_V4.sch (EAGLE design)
At the start: 143 parts, among them IC1 IS25LP080D-JULE-TR_IS25LP080D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, IC3 KSZ9131RNXI-TR, J1 0826-1X1T-KL-F_0826-1X1T-KL-F, J3 ESHF-110-01-L-D-TH, U1 AG9900_AG9905LP, U10 ST-MICROELECTRONICS2_ST1S06PUR, U2 AR8035_AR8035-AL1A-R, U3 XE216-512-TQ128-C20_XE216-512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, U4 ADM1085AKSZ-REEL7_ADM1085AKSZ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, U5 NC7WZ07P6X_NC7WZ07P6X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

Commit message: resolved DRC errors and exported manufacturing data for V4.
Parts:
- removed IC3: KSZ9131RNXI-TR, KSZ9131RNXI-TR:KSZ9131RNXI-TR
- removed R19: 43R2, xmos_avb_brd_V4:RCL_R-EU_R0402
Connections:
- removed net USB_DM_N: J3.20, U3.USB_DM
- removed net USB_DP_P: J3.19, U3.USB_DP
- removed net USB_ID: J3.17, U3.USB_ID
- removed net USB_RTUNE: R19.2, U3.USB_RTUNE
- removed net USB_VBUS: J3.16, U3.USB_VBUS
- net GND: no longer R19.1
Changed lines of the file:
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@@
 </part>
 <part name="FL4" library="xmos_avb_brd_V4" deviceset="BLM21AG471SN1D_BLM21AG471SN1D" device=""/>
-<part name="R19" library="xmos_avb_brd_V4" deviceset="RCL_R-EU_" device="R0402" value="43R2">
-<attribute name="DNP" value="DNP"/>
-</part>
-<part name="SUPPLY24" library="xmos_avb_brd_V4" deviceset="SUPPLY2_GND" device=""/>
 <part name="C24" library="xmos_avb_brd_V4" deviceset="RCL_C-EU" device="C0402" value="100n"/>
 <part name="FL2" library="xmos_avb_brd_V4" deviceset="BLM21PG331SN1D_BLM21PG331SN1D" device=""/>
@@
 <part name="FRAME4" library="xmos_avb_brd_V4" deviceset="FRAMES_A3L-LOC" device=""/>
 <part name="FRAME1" library="xmos_avb_brd_V4" deviceset="FRAMES_A3L-LOC" device=""/>
-<part name="IC3" library="KSZ9131RNXI-TR" deviceset="KSZ9131RNXI-TR" device=""/>
 <part name="J3" library="ESHF-110-01-L-D-TH" deviceset="ESHF-110-01-L-D-TH" device=""/>
 <part name="SUPPLY27" library="xmos_avb_brd_V4" deviceset="SUPPLY2_GND" device=""/>
@@
 <attribute name="NAME" x="365.76" y="-209.042" size="1.524" layer="95"/>
 </instance>
-<instance part="R19" gate="G$1" x="101.6" y="-71.12" smashed="yes">
-<attribute name="NAME" x="97.79" y="-69.6214" size="1.778" layer="95"/>
-<attribute name="VALUE" x="97.79" y="-74.422" size="1.778" layer="96"/>
-<attribute name="DNP" x="104.14" y="-68.58" size="1.778" layer="96"/>
-</instance>
-<instance part="SUPPLY24" gate="GND" x="96.52" y="-76.2" smashed="yes">
-<attribute name="VALUE" x="94.615" y="-79.375" size="1.778" layer="96"/>
-</instance>
 <instance part="C24" gate="G$1" x="63.5" y="-91.44" smashed="yes">
 <attribute name="NAME" x="65.024" y="-91.059" size="1.778" layer="95"/>
@@
 <pinref part="SUPPLY35" gate="GND" pin="GND"/>
 <wire x1="325.12" y1="-101.6" x2="325.12" y2="-96.52" width="0.1524" layer="91"/>
+<pinref part="IC1" gate="G$1" pin="GND"/>
 <wire x1="325.12" y1="-96.52" x2="325.12" y2="-93.98" width="0.1524" layer="91"/>
-<wire x1="320.04" y1="-96.52" x2="325.12" y2="-96.52" width="0.1524" layer="91"/>
+<wire x1="317.98" y1="-96.5" x2="317.98" y2="-96.52" width="0.1524" layer="91"/>
+<wire x1="317.98" y1="-96.52" x2="325.12" y2="-96.52" width="0.1524" layer="91"/>
 <junction x="325.12" y="-96.52"/>
 </segment>
@@
 </segment>
 <segment>
-<pinref part="R19" gate="G$1" pin="1"/>
-<pinref part="SUPPLY24" gate="GND" pin="GND"/>
-<wire x1="96.52" y1="-71.12" x2="96.52" y2="-73.66" width="0.1524" layer="91"/>
-</segment>
-<segment>
-<pinref part="IC1" gate="G$1" pin="GND"/>
-<wire x1="317.98" y1="-96.5" x2="320.04" y2="-96.5" width="0.1524" layer="91"/>
-</segment>
-<segment>
 <pinref part="J3" gate="G$1" pin="3"/>
 <wire x1="241.3" y1="-12.7" x2="213.36" y2="-12.7" width="0.1524" layer="91"/>
@@
 </segment>
 </net>
-<net name="USB_DM_N" class="2">
-<segment>
-<pinref part="U3" gate="G$1" pin="USB_DM"/>
-<wire x1="134.62" y1="-63.5" x2="121.92" y2="-63.5" width="0.1524" layer="91"/>
-<label x="121.92" y="-63.5" size="1.778" layer="95"/>
-</segment>
-<segment>
-<wire x1="284.48" y1="-33.02" x2="264.16" y2="-33.02" width="0.1524" layer="91"/>
-<label x="266.7" y="-33.02" size="1.778" layer="95"/>
-<pinref part="J3" gate="G$1" pin="20"/>
-</segment>
-</net>
-<net name="USB_DP_P" class="2">
-<segment>
-<pinref part="U3" gate="G$1" pin="USB_DP"/>
-<wire x1="134.62" y1="-66.04" x2="121.92" y2="-66.04" width="0.1524" layer="91"/>
-<label x="121.92" y="-66.04" size="1.778" layer="95"/>
-</segment>
-<segment>
-<wire x1="241.3" y1="-33.02" x2="220.98" y2="-33.02" width="0.1524" layer="91"/>
-<label x="220.98" y="-33.02" size="1.778" layer="95"/>
-<pinref part="J3" gate="G$1" pin="19"/>
-</segment>
-</net>
-<net name="USB_ID" class="0">
-<segment>
-<pinref part="U3" gate="G$1" pin="USB_ID"/>
-<wire x1="134.62" y1="-68.58" x2="121.92" y2="-68.58" width="0.1524" layer="91"/>
-<label x="121.92" y="-68.58" size="1.778" layer="95"/>
-</segment>
-<segment>
-<wire x1="241.3" y1="-30.48" x2="220.98" y2="-30.48" width="0.1524" layer="91"/>
-<label x="220.98" y="-30.48" size="1.778" layer="95"/>
-<pinref part="J3" gate="G$1" pin="17"/>
-</segment>
-</net>
-<net name="USB_VBUS" class="0">
-<segment>
-<pinref part="U3" gate="G$1" pin="USB_VBUS"/>
-<wire x1="134.62" y1="-73.66" x2="121.92" y2="-73.66" width="0.1524" layer="91"/>
-<label x="121.92" y="-73.66" size="1.778" layer="95"/>
-</segment>
-<segment>
-<wire x1="284.48" y1="-27.94" x2="264.16" y2="-27.94" width="0.1524" layer="91"/>
-<label x="279.4" y="-27.94" size="1.778" layer="95"/>
-<pinref part="J3" gate="G$1" pin="16"/>
-</segment>
-</net>
-<net name="USB_RTUNE" class="0">
-<segment>
-<pinref part="U3" gate="G$1" pin="USB_RTUNE"/>
-<wire x1="134.62" y1="-71.12" x2="106.68" y2="-71.12" width="0.1524" layer="91"/>
-<label x="121.92" y="-71.12" size="1.778" layer="95"/>
-<pinref part="R19" gate="G$1" pin="2"/>
-<wire x1="114.3" y1="-71.12" x2="106.68" y2="-71.12" width="0.1524" layer="91"/>
-</segment>
-</net>
 <net name="X1D37" class="0">
 <segment>
@@
 <attribute name="SHEET" x="352.425" y="-251.46" size="2.54" layer="94"/>
 </instance>
-<instance part="IC3" gate="G$1" x="439.42" y="-149.86" smashed="yes">
-<attribute name="NAME" x="417.83" y="-81.28" size="1.778" layer="95" align="center-left"/>
-<attribute name="VALUE" x="417.83" y="-83.82" size="1.778" layer="96" align="center-left"/>
-</instance>
 </instances>
 <busses>
@@
 <pinref part="J1" gate="G$1" pin="MH2"/>
 <pinref part="R2" gate="G$1" pin="2"/>
-<wire x1="76.2" y1="-160.02" x2="73.66" y2="-160.02" width="0.1524" layer="91"/>
 <wire x1="73.66" y1="-160.02" x2="71.12" y2="-160.02" width="0.1524" layer="91"/>
 </segment>
@@
 </sheet>
 </sheets>
-<errors>
-</errors>
 </schematic>
 </drawing>
